File: imm/imm.kicad_pcb (KiCad board)
At the start: 2 copper layers, 20.3 x 20.3 mm, 15 parts, among them J1 Conn_01x02, J2 Conn_01x03, Q1 D4184, U1 EL817

Commit message: Hmmm
Parts:
- moved D1 17.8 mm to (113.7, 94.0)
- moved R3 11.7 mm to (121.3, 90.8), turned to 180 degrees
- moved R5 8.26 mm to (113.7, 90.8), turned to 0 degrees
- moved D2 7.85 mm to (117.5, 90.8), turned to 0 degrees
- moved R1 3.86 mm to (108.6, 95.2)
- moved Q1 3.81 mm to (116.8, 85.1)
- moved J1 1.27 mm to (108.6, 88.9)
- moved R2 0.90 mm to (117.5, 94.0)
- moved R4 0.63 mm to (121.3, 94.0)
Routing:
- net /LD: track 0.00 -> 23.4 mm
- net Net-(Q1-Pad1): track 0.00 -> 11.9 mm
- net GND1: track 0.00 -> 9.75 mm
- net Net-(D1-Pad1): track 0.00 -> 9.70 mm
- net VDC: track 0.00 -> 7.62 mm
- net Net-(R3-Pad1): track 0.00 -> 6.96 mm
- net Net-(J1-Pad1): track 0.00 -> 6.93 mm
- net Net-(R1-Pad2): track 0.00 -> 3.45 mm
- net Net-(D2-Pad1): track 0.00 -> 2.20 mm
- removed copper zone on F.Cu, net /LD
- removed copper zone on B.Cu, net GND1
- removed copper zone on F.Cu, net GND1
Other:
- board text added: "+V"
- board text added: "GND"
- board text added: "LOAD"
- board text added: "PWM"

Commit message: Tweaking
Parts:
- removed D1: 1N4148, Diode_SMD:D_SOD-323
- Q1: footprint Package_TO_SOT_SMD:TO-252-3_TabPin2 -> Package_TO_SOT_SMD:TO-252-2
- moved R1 5.24 mm to (113.7, 94.0)
- moved J1 1.27 mm to (108.6, 90.2)
Routing:
- net /LD: track 23.4 -> 32.9 mm, vias 0 -> 5
- net Net-(R2-Pad2): track 9.70 -> 7.77 mm
- net GND1: track 9.75 -> 8.43 mm
- net Net-(R1-Pad2): track 3.45 -> 4.18 mm
- net Net-(R3-Pad1): track 6.96 -> 6.28 mm
- net GND2: vias 0 -> 10
- added copper zone on F.Cu, net /LD
Other:
- board text added: "${TITLE} rev. ${REVISION}"
- board text added: "6-30V"
