File: imm/imm.kicad_sch (KiCad schematic)
At the start: 15 parts, among them J1 Conn_01x02, J2 Conn_01x03, Q1 D4184, U1 EL817

Commit message: Hmmm
Other:
- moved on the sheet: D1, D2, H1, H2, H3, H4, J1, J2, Q1, R1, R2, R3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

Commit message: Tweaking
Parts:
- removed D1: 1N4148, Diode_SMD:D_SOD-323, symbol Device:D
- Q1: footprint Package_TO_SOT_SMD:TO-252-3_TabPin2 -> Package_TO_SOT_SMD:TO-252-2
Other:
- company: (none) -> ${URL}
- title: (none) -> ${TITLE}
- moved on the sheet: D2, J1, J2, Q1, R1, R2, R3, R4, R5, U1
